File: hardware/record.brd (EAGLE design)
At the start: 34 x 34 mm, 24 parts, among them U1 MAX9939, U2 CBRHDSH1-40L, U3 MSP430FR5728_RGE_24, U4 FDG6303N, U5 FDG6303N

Commit message: Final demo for California. Everything works well. Four nodes stress test worked great. Not awesome with quick changing energy harvesters like piezo though.
Parts:
- R1: value 33k -> 47k
Changed lines of the file:
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@@
 <attribute name="PROD_ID" value="CAP-08064" x="6.7" y="8.7" size="1.778" layer="27" rot="R90" display="off"/>
 </element>
-<element name="R1" library="SparkFun-Resistors" package="0805" value="33k" x="8" y="4.4" rot="R270">
+<element name="R1" library="SparkFun-Resistors" package="0805" value="47k" x="8" y="4.4" rot="R270">
 <attribute name="PROD_ID" value="RES-09883" x="8" y="4.4" size="1.778" layer="27" rot="R270" display="off"/>
 </element>
