File: hardware/record_revc_ina225.sch (EAGLE design)
At the start: 34 parts, among them IC1 CC1101, U1 INA225, U2 CBRHDSH1-40L, U3 MSP430FR5728_RGE_24, U4 FDG6303N, U5 FDG6303N, U6 0896BM15A0001, X1 NX3225GA-26.000M-STD-CRG-2

Commit message: Final hardware for circuit hub
Parts:
- R4: value (none) -> 200
- R6: value (none) -> 10k
- R7: value (none) -> 100k
- R8: value (none) -> 1M
Changed lines of the file:
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@@
 <part name="GND4" library="SparkFun-Aesthetics" deviceset="GND" device=""/>
 <part name="GND5" library="SparkFun-Aesthetics" deviceset="GND" device=""/>
-<part name="R4" library="SparkFun-Resistors" deviceset="0.22OHM1/4W1%(0805)" device=""/>
-<part name="R6" library="SparkFun-Resistors" deviceset="0.22OHM1/4W1%(0805)" device=""/>
-<part name="R7" library="SparkFun-Resistors" deviceset="0.22OHM1/4W1%(0805)" device=""/>
-<part name="R8" library="SparkFun-Resistors" deviceset="0.22OHM1/4W1%(0805)" device=""/>
+<part name="R4" library="SparkFun-Resistors" deviceset="0.22OHM1/4W1%(0805)" device="" value="200"/>
+<part name="R6" library="SparkFun-Resistors" deviceset="0.22OHM1/4W1%(0805)" device="" value="10k"/>
+<part name="R7" library="SparkFun-Resistors" deviceset="0.22OHM1/4W1%(0805)" device="" value="100k"/>
+<part name="R8" library="SparkFun-Resistors" deviceset="0.22OHM1/4W1%(0805)" device="" value="1M"/>
 <part name="GND9" library="SparkFun-Aesthetics" deviceset="GND" device=""/>
 <part name="GND12" library="SparkFun-Aesthetics" deviceset="GND" device=""/>
